File: _autosave-merchants 60.kicad_pcb (KiCad board)
At the start: 4 copper layers, 304.8 x 122.2 mm, 182 parts, among them SW1 SW_PUSH, U1 ATmega32U4-AU, Y1 16MHz

Commit message: Finalising PCB and Generating Gerbers
Routing:
- net col9: track 281.0 -> 276.5 mm, vias 1 -> 3
- net +5V: track 77.8 -> 81.1 mm, vias 6 -> 7
- net Net-(C5-Pad2): track 7.56 -> 8.34 mm
- net Net-(C4-Pad1): track 8.45 -> 9.04 mm
- net GND: track 282.8 -> 283.3 mm
- net D+: track 160.2 -> 160.8 mm
- net D-: track 159.1 -> 159.7 mm
- net VCC: track 150.8 -> 151.4 mm
Other:
- board size 304.8 x 122.2 mm -> 304.8 x 123.8 mm

Commit message: Converting the PCB from 4 layer to 2 layer
Im fucking retarded but I'm also a fucking god
Connections:
- U1 pad 27: row5 -> row3
- U1 pad 29: row3 -> row5
Routing:
- net col10: track 288.2 -> 350.9 mm, vias 1 -> 5
- net col11: track 319.4 -> 371.3 mm, vias 1 -> 7
- net col0: track 163.3 -> 120.7 mm, vias 1 -> 0
- net VCC: track 151.4 -> 185.5 mm, vias 2 -> 3
- net row2: track 314.6 -> 348.0 mm, vias 1 -> 2
- net col8: track 231.5 -> 260.1 mm, vias 1 -> 3
- net col15: track 459.2 -> 431.2 mm, vias 1 -> 3
- net col7: track 211.6 -> 238.8 mm, vias 1 -> 6
- net col12: track 343.8 -> 366.8 mm, vias 1 -> 3
- net col14: track 424.8 -> 403.1 mm, vias 1 -> 3
- net D+: track 160.8 -> 182.1 mm, vias 2 -> 1
- net col9: track 276.5 -> 296.6 mm
- net D-: track 159.7 -> 179.8 mm, vias 2 -> 1
- net row1: track 317.6 -> 335.3 mm, vias 1 -> 2
- net col3: track 143.5 -> 130.6 mm, vias 1 -> 3
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Other:
- copper layers 4 -> 2
